File: i2s_soundcard.sch (KiCad schematic (older format))
At the start: 13 parts, among them J1 Conn_01x08, J2 Conn_01x06, J3 Conn_01x05, J4 Conn_01x11, J5 Conn_01x04, U1 TLV320AIC3104IRHBT, U6 TLV7111830DSER, U7 TPD4E02B04DQAR, U8 TPD4E02B04DQAR

Commit message: Tidy up schematic a bit
Connections:
- net detect?: now reaches J1.7 (Pin_7), U8.4 (D2+), U8.7 (NC)
Changed lines of the file:
@@
 EELAYER 30 0
 EELAYER END
-$Descr A4 11693 8268
+$Descr B 17000 11000
 encoding utf-8
 Sheet 1 3
@@
 P 4350 1550
 F 0 "U1" V 4550 1550 60  0000 C CNN
-F 1 "TLV320AIC3104IRHBT" V 4700 1350 60  0000 C CNN
+F 1 "TLV320AIC3104IRHBT" V 4700 1550 60  0000 C CNN
 F 2 "footprints:TLV320AIC3104IRHBT" H 5950 1790 60  0001 C CNN
 F 3 "" H 4350 1550 60  0000 C CNN
@@
 U 1 1 602C8967
 P 1200 750
-F 0 "U6" H 2000 1137 60  0000 C CNN
-F 1 "TLV7111830DSER" H 2000 1031 60  0000 C CNN
+F 0 "U6" H 2000 400 60  0000 C CNN
+F 1 "TLV7111830DSER" H 2000 250 60  0000 C CNN
 F 2 "footprints:TLV7111830DSER" H 2000 990 60  0001 C CNN
 F 3 "" H 1200 750 60  0000 C CNN
@@
 U 1 1 602651EC
 P 4450 3850
-F 0 "U1" V 4700 3100 60  0000 L CNN
-F 1 "TLV320AIC3104IRHBT" V 4850 3100 60  0000 L CNN
+F 0 "U1" H 4350 4000 60  0000 L CNN
+F 1 "TLV320AIC3104IRHBT" H 4000 4300 60  0000 L CNN
 F 2 "footprints:TLV320AIC3104IRHBT" H 6050 4090 60  0001 C CNN
 F 3 "" H 4450 3850 60  0000 C CNN
@@
 Text Label 2450 2850 0    50   ~ 0
 ~shutdown
-Text Label 2650 3150 0    50   ~ 0
+Text Label 2600 3150 0    50   ~ 0
 reset
 Wire Wire Line
@@
 Wire Wire Line
 	2600 3150 2450 3150
-Wire Wire Line
-	2650 3150 2600 3150
-Connection ~ 2600 3150
 Wire Wire Line
 	1750 2750 1750 2450
@@
 Connection ~ 6950 5500
 Connection ~ 8350 5500
+Text Label 6850 6100 2    50   ~ 0
+detect?
 $EndSCHEMATC
