File: i2s_soundcard.sch (KiCad schematic (older format))
At the start: 19 parts, among them J1 Conn_01x08, J2 Conn_01x06, J3 Conn_01x04, J4 Conn_01x11, J5 Conn_01x03, U1 TLV320AIC3104IRHBT, U6 TLV7111830DSER, U7 TPD4E02B04DQAR, U8 TPD4E02B04DQAR

Commit message: Change C2/C3 to 1206, adjust board to make that fit. Add courtyard to ESD protection diodes
Parts:
- C2, C3: footprint Capacitor_SMD:C_0402_1005Metric -> Capacitor_SMD:C_1206_3216Metric
Changed lines of the file:
@@
 F 0 "C3" V 6148 3550 50  0000 C CNN
 F 1 "220uF" V 6250 3550 50  0000 C CNN
-F 2 "Capacitor_SMD:C_0402_1005Metric" H 6438 3400 50  0001 C CNN
+F 2 "Capacitor_SMD:C_1206_3216Metric" H 6438 3400 50  0001 C CNN
 F 3 "~" H 6400 3550 50  0001 C CNN
 	1    6400 3550
@@
 F 0 "C2" V 6148 3350 50  0000 C CNN
 F 1 "220uF" V 6239 3350 50  0000 C CNN
-F 2 "Capacitor_SMD:C_0402_1005Metric" H 6438 3200 50  0001 C CNN
+F 2 "Capacitor_SMD:C_1206_3216Metric" H 6438 3200 50  0001 C CNN
 F 3 "~" H 6400 3350 50  0001 C CNN
 	1    6400 3350
