File: als.kicad_sch (KiCad schematic)
At the start: 3 parts, among them J11 Conn_02x12_Odd_Even, U14 TCA9802, U16 MIC5365-3.0YD5-TR

Commit message: Final touches on Radxa CM3 version of the board
Parts:
- added C4, C5, C6, C7: 1uF, Capacitor_SMD:C_0402_1005Metric, symbol Device:C
Connections:
- net GND: now also C4.2, C5.2, C6.2, C7.2
- net VCC_3.0: now also C5.1, C7.1
- net VCC_3.3: now also C6.1; no longer U16.3 (EN), U16.4 (VIN)
- new net VBAT_3.7: C4.1, U16.3 (EN), U16.4 (VIN)
Changed lines of the file:
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@@
   (junction (at 128.27 105.41) (diameter 1.016) (color 0 0 0 0)
   )
+  (junction (at 113.03 63.5) (diameter 0) (color 0 0 0 0)
+  )
   (junction (at 140.97 92.71) (diameter 1.016) (color 0 0 0 0)
   )
+  (junction (at 100.33 27.94) (diameter 0) (color 0 0 0 0)
+  )
   (junction (at 128.27 102.87) (diameter 1.016) (color 0 0 0 0)
   )
@@
   (junction (at 128.27 100.33) (diameter 1.016) (color 0 0 0 0)
   )
+  (junction (at 105.41 27.94) (diameter 0) (color 0 0 0 0)
+  )
   (junction (at 128.27 97.79) (diameter 1.016) (color 0 0 0 0)
   )
@@
   )
   (junction (at 128.27 95.25) (diameter 1.016) (color 0 0 0 0)
+  )
+  (junction (at 78.74 63.5) (diameter 0) (color 0 0 0 0)
   )
   (no_connect (at 88.9 85.09))
@@
     (stroke (width 0) (type solid) (color 0 0 0 0))
   )
+  (wire (pts (xy 78.74 63.5) (xy 73.66 63.5))
+    (stroke (width 0) (type default) (color 0 0 0 0))
+  )
   (wire (pts (xy 142.24 83.82) (xy 140.97 82.55))
     (stroke (width 0) (type solid) (color 0 0 0 0))
   )
+  (wire (pts (xy 105.41 27.94) (xy 105.41 43.18))
+    (stroke (width 0) (type default) (color 0 0 0 0))
+  )
   (wire (pts (xy 128.27 85.09) (xy 128.27 87.63))
     (stroke (width 0) (type solid) (color 0 0 0 0))
@@
     (stroke (width 0) (type solid) (color 0 0 0 0))
   )
+  (wire (pts (xy 96.52 63.5) (xy 78.74 63.5))
+    (stroke (width 0) (type default) (color 0 0 0 0))
+  )
+  (wire (pts (xy 101.6 63.5) (xy 101.6 69.85))
+    (stroke (width 0) (type default) (color 0 0 0 0))
+  )
   (wire (pts (xy 140.97 90.17) (xy 140.97 92.71))
     (stroke (width 0) (type solid) (color 0 0 0 0))
@@
     (stroke (width 0) (type solid) (color 0 0 0 0))
   )
+  (wire (pts (xy 113.03 63.5) (xy 101.6 63.5))
+    (stroke (width 0) (type default) (color 0 0 0 0))
+  )
+  (wire (pts (xy 134.62 27.94) (xy 147.32 27.94))
+    (stroke (width 0) (type default) (color 0 0 0 0))
+  )
   (wire (pts (xy 109.22 82.55) (xy 128.27 82.55))
     (stroke (width 0) (type solid) (color 0 0 0 0))
@@
     (stroke (width 0) (type solid) (color 0 0 0 0))
   )
-  (wire (pts (xy 105.41 27.94) (xy 105.41 43.18))
+  (wire (pts (xy 115.57 63.5) (xy 113.03 63.5))
+    (stroke (width 0) (type default) (color 0 0 0 0))
+  )
+  (wire (pts (xy 100.33 27.94) (xy 105.41 27.94))
     (stroke (width 0) (type solid) (color 0 0 0 0))
   )
   (wire (pts (xy 116.84 27.94) (xy 105.41 27.94))
+    (stroke (width 0) (type solid) (color 0 0 0 0))
+  )
+  (wire (pts (xy 96.52 69.85) (xy 96.52 63.5))
+    (stroke (width 0) (type default) (color 0 0 0 0))
+  )
+  (wire (pts (xy 96.52 27.94) (xy 100.33 27.94))
     (stroke (width 0) (type solid) (color 0 0 0 0))
   )
@@
     (effects (font (size 1.27 1.27)) (justify left bottom))
   )
-  (label "VCC_3.0" (at 101.6 69.85 0)
+  (label "VCC_3.0" (at 115.57 63.5 0)
     (effects (font (size 1.27 1.27)) (justify left bottom))
   )
@@
     (effects (font (size 1.27 1.27)) (justify right))
   )
-  (hierarchical_label "VCC_3.3" (shape input) (at 105.41 27.94 180)
+  (hierarchical_label "VBAT_3.7" (shape input) (at 96.52 27.94 180)
     (effects (font (size 1.27 1.27)) (justify right))
   )
@@
     (effects (font (size 1.27 1.27)) (justify right))
   )
-  (hierarchical_label "VCC_3.3" (shape input) (at 96.52 69.85 180)
+  (hierarchical_label "VCC_3.3" (shape input) (at 73.66 63.5 180)
     (effects (font (size 1.27 1.27)) (justify right))
+  )
+  (symbol (lib_id "Device:C") (at 100.33 31.75 0) (unit 1)
+    (in_bom yes) (on_board yes) (fields_autoplaced)
+    (property "Reference" "C4" (id 0) (at 103.251 30.8415 0)
+      (effects (font (size 1.27 1.27)) (justify left))
+    )
+    (property "Value" "1uF" (id 1) (at 103.251 33.6166 0)
+      (effects (font (size 1.27 1.27)) (justify left))
+    )
+    (property "Footprint" "Capacitor_SMD:C_0402_1005Metric" (id 2) (at 101.2952 35.56 0)
+      (effects (font (size 1.27 1.27)) hide)
+    )
+    (property "Datasheet" "~" (id 3) (at 100.33 31.75 0)
+      (effects (font (size 1.27 1.27)) hide)
+    )
+    (pin "1")
+    (pin "2")
   )
   (symbol (lib_id "power:GND") (at 125.73 58.42 0) (unit 1)
@@
     (pin "1")
   )
+  (symbol (lib_id "Device:C") (at 113.03 67.31 0) (unit 1)
+    (in_bom yes) (on_board yes) (fields_autoplaced)
+    (property "Reference" "C7" (id 0) (at 115.951 66.4015 0)
+      (effects (font (size 1.27 1.27)) (justify left))
+    )
+    (property "Value" "1uF" (id 1) (at 115.951 69.1766 0)
+      (effects (font (size 1.27 1.27)) (justify left))
+    )
+    (property "Footprint" "Capacitor_SMD:C_0402_1005Metric" (id 2) (at 113.9952 71.12 0)
+      (effects (font (size 1.27 1.27)) hide)
+    )
+    (property "Datasheet" "~" (id 3) (at 113.03 67.31 0)
+      (effects (font (size 1.27 1.27)) hide)
+    )
+    (pin "1")
+    (pin "2")
+  )
   (symbol (lib_id "power:GND") (at 134.62 111.76 0) (unit 1)
     (in_bom yes) (on_board yes) (fields_autoplaced)
@@
     )
     (pin "1")
+  )
+  (symbol (lib_id "Device:C") (at 78.74 67.31 0) (unit 1)
+    (in_bom yes) (on_board yes) (fields_autoplaced)
+    (property "Reference" "C6" (id 0) (at 81.661 66.4015 0)
+      (effects (font (size 1.27 1.27)) (justify left))
+    )
+    (property "Value" "1uF" (id 1) (at 81.661 69.1766 0)
+      (effects (font (size 1.27 1.27)) (justify left))
+    )
+    (property "Footprint" "Capacitor_SMD:C_0402_1005Metric" (id 2) (at 79.7052 71.12 0)
+      (effects (font (size 1.27 1.27)) hide)
+    )
+    (property "Datasheet" "~" (id 3) (at 78.74 67.31 0)
+      (effects (font (size 1.27 1.27)) hide)
+    )
+    (pin "1")
+    (pin "2")
   )
   (symbol (lib_id "power:GND") (at 99.06 95.25 0) (unit 1)
@@
     (pin "9")
   )
+  (symbol (lib_id "power:GND") (at 78.74 71.12 0) (unit 1)
+    (in_bom yes) (on_board yes) (fields_autoplaced)
+    (property "Reference" "#PWR0121" (id 0) (at 78.74 77.47 0)
+      (effects (font (size 1.27 1.27)) hide)
+    )
+    (property "Value" "GND" (id 1) (at 78.74 75.6825 0))
+    (property "Footprint" "" (id 2) (at 78.74 71.12 0)
+      (effects (font (size 1.27 1.27)) hide)
+    )
+    (property "Datasheet" "" (id 3) (at 78.74 71.12 0)
+      (effects (font (size 1.27 1.27)) hide)
+    )
+    (pin "1")
+  )
+  (symbol (lib_id "power:GND") (at 147.32 35.56 0) (unit 1)
+    (in_bom yes) (on_board yes) (fields_autoplaced)
+    (property "Reference" "#PWR0117" (id 0) (at 147.32 41.91 0)
+      (effects (font (size 1.27 1.27)) hide)
+    )
+    (property "Value" "GND" (id 1) (at 147.32 39.8844 0))
+    (property "Footprint" "" (id 2) (at 147.32 35.56 0)
+      (effects (font (size 1.27 1.27)) hide)
+    )
+    (property "Datasheet" "" (id 3) (at 147.32 35.56 0)
+      (effects (font (size 1.27 1.27)) hide)
+    )
+    (pin "1")
+  )
   (symbol (lib_id "Interface:TCA9802") (at 99.06 82.55 0) (unit 1)
     (in_bom yes) (on_board yes)
@@
     (pin "8")
   )
+  (symbol (lib_id "Device:C") (at 147.32 31.75 0) (unit 1)
+    (in_bom yes) (on_board yes) (fields_autoplaced)
+    (property "Reference" "C5" (id 0) (at 150.241 30.8415 0)
+      (effects (font (size 1.27 1.27)) (justify left))
+    )
+    (property "Value" "1uF" (id 1) (at 150.241 33.6166 0)
+      (effects (font (size 1.27 1.27)) (justify left))
+    )
+    (property "Footprint" "Capacitor_SMD:C_0402_1005Metric" (id 2) (at 148.2852 35.56 0)
+      (effects (font (size 1.27 1.27)) hide)
+    )
+    (property "Datasheet" "~" (id 3) (at 147.32 31.75 0)
+      (effects (font (size 1.27 1.27)) hide)
+    )
+    (pin "1")
+    (pin "2")
+  )
+  (symbol (lib_id "power:GND") (at 113.03 71.12 0) (unit 1)
+    (in_bom yes) (on_board yes) (fields_autoplaced)
+    (property "Reference" "#PWR0118" (id 0) (at 113.03 77.47 0)
+      (effects (font (size 1.27 1.27)) hide)
+    )
+    (property "Value" "GND" (id 1) (at 113.03 75.6825 0))
+    (property "Footprint" "" (id 2) (at 113.03 71.12 0)
+      (effects (font (size 1.27 1.27)) hide)
+    )
+    (property "Datasheet" "" (id 3) (at 113.03 71.12 0)
+      (effects (font (size 1.27 1.27)) hide)
+    )
+    (pin "1")
+  )
   (symbol (lib_id "MIC5365-3.0YD5-TR:MIC5365-3.0YD5-TR") (at 105.41 40.64 0) (unit 1)
-    (in_bom yes) (on_board yes) (fields_autoplaced)
+    (in_bom yes) (on_board yes)
     (property "Reference" "U16" (id 0) (at 139.1285 42.2924 0)
       (effects (font (size 1.524 1.524)) (justify left))
@@
       (effects (font (size 1.524 1.524)) hide)
     )
-    (property "Datasheet" "" (id 3) (at 105.41 40.64 0)
-      (effects (font (size 1.524 1.524)))
+    (property "Datasheet" "${KIPRJMOD}/datasheets/mic5365.pdf" (id 3) (at 107.95 52.07 0)
+      (effects (font (size 1.524 1.524)) hide)
     )
     (pin "1")
@@
     (pin "5")
   )
+  (symbol (lib_id "power:GND") (at 100.33 35.56 0) (unit 1)
+    (in_bom yes) (on_board yes) (fields_autoplaced)
+    (property "Reference" "#PWR0116" (id 0) (at 100.33 41.91 0)
+      (effects (font (size 1.27 1.27)) hide)
+    )
+    (property "Value" "GND" (id 1) (at 100.33 39.8844 0))
+    (property "Footprint" "" (id 2) (at 100.33 35.56 0)
+      (effects (font (size 1.27 1.27)) hide)
+    )
+    (property "Datasheet" "" (id 3) (at 100.33 35.56 0)
+      (effects (font (size 1.27 1.27)) hide)
+    )
+    (pin "1")
+  )
 )
