File: gt9113_breakout.kicad_sch (KiCad schematic)
At the start: 10 parts, among them J6 504740-5100, J7 504740-5100, U9 GT9113

Commit message: Lots more work on the cm3 version of this board.
Connections:
- net AVDD18: now reaches C26.1, U9.24 (AVDD18)
- net DVDD12: now reaches C25.1, U9.25 (DVDD12)
Changed lines of the file:
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@@
     (effects (font (size 1.27 1.27)) (justify right bottom))
+  )
+  (label "DVDD12" (at 264.16 29.21 0)
+    (effects (font (size 1.27 1.27)) (justify left bottom))
   )
   (label "X2" (at 191.77 289.56 270)
@@
     (effects (font (size 1.27 1.27)) (justify left bottom))
   )
+  (label "AVDD28" (at 264.16 24.13 0)
+    (effects (font (size 1.27 1.27)) (justify left bottom))
+  )
   (label "Y8" (at 111.76 289.56 270)
     (effects (font (size 1.27 1.27)) (justify right bottom))
@@
     (effects (font (size 1.27 1.27)) (justify left bottom))
   )
+  (label "AVDD18" (at 264.16 26.67 0)
+    (effects (font (size 1.27 1.27)) (justify left bottom))
+  )

Commit message: Final touches on Radxa CM3 version of the board
Connections:
- net GND: now also U9.89 (PAD)
- net Sensor_OPT1: now reaches R13.2, U9.28 (Sensor_OPT1)
- net Sensor_OPT2: now reaches R11.1, R12.2, U9.29 (Sensor_OPT2)
Changed lines of the file:
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@@
+    (effects (font (size 1.27 1.27)) (justify left bottom))
+  )
+  (label "Sensor_OPT1" (at 217.17 142.24 0)
     (effects (font (size 1.27 1.27)) (justify left bottom))
   )
@@
   (label "Y27" (at 173.99 289.56 270)
     (effects (font (size 1.27 1.27)) (justify right bottom))
+  )
+  (label "Sensor_OPT2" (at 217.17 139.7 0)
+    (effects (font (size 1.27 1.27)) (justify left bottom))
   )
   (label "Y14" (at 347.98 289.56 270)
@@
     (pin "88")
     (pin "9")
+    (pin "89")
   )
   (symbol (lib_id "Device:C") (at 283.21 33.02 0) (unit 1)
@@
     (pin "2")
   )
+  (symbol (lib_id "power:GND") (at 242.57 237.49 0) (unit 1)
+    (in_bom yes) (on_board yes)
+    (property "Reference" "#PWR0115" (id 0) (at 242.57 243.84 0)
+      (effects (font (size 1.27 1.27)) hide)
+    )
+    (property "Value" "GND" (id 1) (at 242.697 241.8842 0))
+    (property "Footprint" "" (id 2) (at 242.57 237.49 0)
+      (effects (font (size 1.27 1.27)) hide)
+    )
+    (property "Datasheet" "" (id 3) (at 242.57 237.49 0)
+      (effects (font (size 1.27 1.27)) hide)
+    )
+    (pin "1")
+  )
   (sheet_instances
